Commit message: lettura joints
tramite /ros2 topic echo /dynamic..

File: urdf/common.gazebo.xacro (robot description, xacro)
@@ -1,23 +1,3 @@
 <?xml version="1.0"?>
 <robot xmlns:xacro="http://wiki.ros.org/xacro">
-  <gazebo>
-    <plugin name="ros_control" filename="libgazebo_ros_control.so">
-      <!--robotNamespace>/</robotNamespace-->
-      <!--robotSimType>gazebo_ros_control/DefaultRobotHWSim</robotSimType-->
-    </plugin>
-<!--
-    <plugin name="gazebo_ros_power_monitor_controller" filename="libgazebo_ros_power_monitor.so">
-      <alwaysOn>true</alwaysOn>
-      <updateRate>1.0</updateRate>
-      <timeout>5</timeout>
-      <powerStateTopic>power_state</powerStateTopic>
-      <powerStateRate>10.0</powerStateRate>
-      <fullChargeCapacity>87.78</fullChargeCapacity>
-      <dischargeRate>-474</dischargeRate>
-      <chargeRate>525</chargeRate>
-      <dischargeVoltage>15.52</dischargeVoltage>
-      <chargeVoltage>16.41</chargeVoltage>
-    </plugin>
--->
-  </gazebo>
 </robot>

File: urdf/tm.gazebo.xacro (robot description, xacro)
@@ -20,9 +20,4 @@
       <selfCollide>true</selfCollide>
     </gazebo>
-    <!--
-    <gazebo reference="${prefix}ee_link">
-      <selfCollide>true</selfCollide>
-    </gazebo>
-    -->
   </xacro:macro>
 </robot>

File: urdf/tm5_900.urdf.xacro (robot description, xacro)
@@ -42,14 +42,4 @@
     <!-- Kinematic model -->
     <!-- Properties from tmcontrol.conf -->
-    <!--
-      DH for TM5-900:
-      a = [0.0000, 0.4290, 0.4115,  0.0000,  0.0000,  0.0000]
-      d = [0.1452,  0.0000,  0.0000,  -0.1223,  0.1060,  0.11315]
-      alpha = [-0.5*pi, 0, 0, 0.5*pi, 0.5*pi, 0]
-      q_home_offset = [0, -0.5*pi, 0, 0.5*pi, 0, 0]
-      joint_direction = [-1, -1, 1, -1, 1, 1]
-      mass = [4.5, 10.5, 2.1, 1.45, 1.45, 0.4]
-      center_of_mass = [ [0, -0.02561, 0.00193], [0.2125, 0, 0.11336], [0.11993, 0.0, 0.0265], [0, -0.0018, 0.01634], [0, 0.0018,0.01634], [0, 0, -0.001159] ](tm900)
-    -->
     <xacro:property name="tm_d1" value="0.1452" />
     <xacro:property name="tm_a2" value="0.4290" />

File: urdf/tm5_900_robot.urdf.xacro (robot description, xacro)
@@ -16,3 +16,22 @@
     <origin xyz="0 0 0" rpy="0 0 0" />
   </joint>
+  <ros2_control name="GazeboSystem" type="system">
+    <hardware>
+      <plugin>gazebo_ros2_control/GazeboSystem</plugin>
+    </hardware>
+    <joint name="shoulder_1_joint">
+      <command_interface name="position" />
+      <state_interface name="position" />
+    </joint>
+    <joint name="shoulder_2_joint">
+      <command_interface name="velocity" />
+      <state_interface name="velocity" />
+      <state_interface name="position" />
+    </joint>
+  </ros2_control>
+  <gazebo>
+    <plugin filename="libgazebo_ros2_control.so" name="gazebo_ros2_control">
+      <parameters>$(find my_robot_gazebo)/config/prova.yaml</parameters>
+    </plugin>
+  </gazebo>
 </robot>
