Commit message: provvisorio

File: urdf/tm5_900_robot.urdf.xacro (robot description, xacro)
@@ -27,7 +27,32 @@
     </joint>
     <joint name="shoulder_2_joint">
-      <command_interface name="velocity" />
+      <command_interface name="position" />
+      <state_interface name="position" />
+      <state_interface name="velocity" />
+      <state_interface name="effort" />
+    </joint>
+    <joint name="elbow_joint">
+      <command_interface name="position" />
+      <state_interface name="position" />
+      <state_interface name="velocity" />
+      <state_interface name="effort" />
+    </joint>
+    <joint name="wrist_1_joint">
+      <command_interface name="position" />
+      <state_interface name="position" />
+      <state_interface name="velocity" />
+      <state_interface name="effort" />
+    </joint>
+    <joint name="wrist_2_joint">
+      <command_interface name="position" />
+      <state_interface name="position" />
+      <state_interface name="velocity" />
+      <state_interface name="effort" />
+    </joint>
+    <joint name="wrist_3_joint">
+      <command_interface name="position" />
       <state_interface name="velocity" />
       <state_interface name="position" />
+      <state_interface name="effort" />
     </joint>
   </ros2_control>
