Commit message: Prima implementazione collisione

File: altri pacchetti/my_doosan_pkg/description/xacro/macro.bumper_config_mod.xacro (robot description, xacro)
@@ -1,24 +1,107 @@
 <?xml version="1.0"?>
 <robot xmlns:xacro="http://www.ros.org/wiki/xacro">
-	<xacro:macro name="bumper_ctr_sensor">
-		<!-- I need this for contact sensor, "bumper sensor"  -->
-		<!-- I create this file in order to detect self-collisions and collisions with the ground  -->
-		<!-- This helps me to detect if the end effect touch the ground so I can reset the environment -->
-		<gazebo reference="link6">
-			<!-- contact sensor -->
-			<sensor name="end_effector_sensor" type="contact">
+	<!-- Macro per sensori di contatto multipli -->
+	<xacro:macro name="multi_contact_sensors">
+		<!-- Sensore su shoulder_1_link -->
+		<gazebo reference="shoulder_1_link">
+			<sensor name="shoulder_1_link_sensor" type="contact">
 				<selfCollide>true</selfCollide>
 				<alwaysOn>true</alwaysOn>
-				<update_rate>50</update_rate>
+				<update_rate>100</update_rate>
 				<contact>
-					<collision>link6_collision</collision>
+					<collision>shoulder_1_collision</collision>
 				</contact>
-				<!-- gazebo plugin -->
-				<plugin name="gazebo_ros_bumper_sensor" filename="libgazebo_ros_bumper.so">
+				<plugin name="bumper_shoulder_1" filename="libgazebo_ros_bumper.so">
 					<ros>
 						<namespace>contact_sensor</namespace>
-						<remapping>bumper_states:=bumper_link6</remapping>
+						<remapping>bumper_states:=bumper_shoulder_1_link</remapping>
 					</ros>
-					<frame_name>link6</frame_name>
+					<frame_name>shoulder_1_link</frame_name>
+				</plugin>
+			</sensor>
+		</gazebo>
+		<!-- Sensore su arm_1_link -->
+		<gazebo reference="arm_1_link">
+			<sensor name="arm_1_link_sensor" type="contact">
+				<selfCollide>true</selfCollide>
+				<alwaysOn>true</alwaysOn>
+				<update_rate>100</update_rate>
+				<contact>
+					<collision>arm_1_link_collision</collision>
+				</contact>
+				<plugin name="bumper_arm_1" filename="libgazebo_ros_bumper.so">
+					<ros>
+						<namespace>contact_sensor</namespace>
+						<remapping>bumper_states:=bumper_arm_1_link</remapping>
+					</ros>
+					<frame_name>arm_1_link</frame_name>
+				</plugin>
+			</sensor>
+		</gazebo>
+		<gazebo reference="arm_2_link">
+			<sensor name="arm_2_link_sensor" type="contact">
+				<selfCollide>true</selfCollide>
+				<alwaysOn>true</alwaysOn>
+				<update_rate>100</update_rate>
+				<contact>
+					<collision>arm_2_link_collision</collision>
+				</contact>
+				<plugin name="bumper_arm_2" filename="libgazebo_ros_bumper.so">
+					<ros>
+						<namespace>contact_sensor</namespace>
+						<remapping>bumper_states:=bumper_arm_2_link</remapping>
+					</ros>
+					<frame_name>arm_2_link</frame_name>
+				</plugin>
+			</sensor>
+		</gazebo>
+		<gazebo reference="wrist_1_link">
+			<sensor name="wrist_1_link_sensor" type="contact">
+				<selfCollide>true</selfCollide>
+				<alwaysOn>true</alwaysOn>
+				<update_rate>100</update_rate>
+				<contact>
+					<collision>wrist_1_link_collision</collision>
+				</contact>
+				<plugin name="bumper_wrist_1" filename="libgazebo_ros_bumper.so">
+					<ros>
+						<namespace>contact_sensor</namespace>
+						<remapping>bumper_states:=bumper_wrist_1_link</remapping>
+					</ros>
+					<frame_name>wrist_1_link</frame_name>
+				</plugin>
+			</sensor>
+		</gazebo>
+		<gazebo reference="wrist_2_link">
+			<sensor name="wrist_2_link_sensor" type="contact">
+				<selfCollide>true</selfCollide>
+				<alwaysOn>true</alwaysOn>
+				<update_rate>100</update_rate>
+				<contact>
+					<collision>wrist_2_link_collision</collision>
+				</contact>
+				<plugin name="bumper_wrist_2" filename="libgazebo_ros_bumper.so">
+					<ros>
+						<namespace>contact_sensor</namespace>
+						<remapping>bumper_states:=bumper_wrist_2_link</remapping>
+					</ros>
+					<frame_name>wrist_2_link</frame_name>
+				</plugin>
+			</sensor>
+		</gazebo>
+		<gazebo reference="wrist_3_link">
+			<sensor name="wrist_3_link_sensor" type="contact">
+				<selfCollide>true</selfCollide>
+				<alwaysOn>true</alwaysOn>
+				<update_rate>100</update_rate>
+				<contact>
+					<collision>wrist_3_link_collision</collision>
+				</contact>
+				<plugin name="bumper_wrist_3" filename="libgazebo_ros_bumper.so">
+					<ros>
+						<namespace>contact_sensor</namespace>
+						<remapping>bumper_states:=bumper_wrist_3_link</remapping>
+					</ros>
+					<frame_name>wrist_3_link</frame_name>
 				</plugin>
 			</sensor>

File: altri pacchetti/my_doosan_pkg/description/xacro/macro.tm5_900.xacro (robot description, xacro)
@@ -358,5 +358,5 @@
     <xacro:dsr_transmission prefix="" hw_interface="hardware_interface/PositionJointInterface" />
     <xacro:dsr_config_coeff />
-    <!--     <xacro:bumper_ctr_sensor /> -->
-  </xacro:macro>
+    <xacro:multi_contact_sensors/>
+    </xacro:macro>
 </robot>
