Commit message: cosi collide con se stesso + lettura angoli in ordine giusta + in input delta angoli e non angoli

File: altri pacchetti/my_doosan_pkg/description/xacro/macro.bumper_config_mod_old.xacro (robot description, xacro)
@@ -1,9 +1,10 @@
 <?xml version="1.0"?>
 <robot xmlns:xacro="http://www.ros.org/wiki/xacro">
-	<!-- Macro per sensori di contatto multipli -->
-	<xacro:macro name="multi_contact_sensors">
-		<!-- Sensore su shoulder_1_link -->
+	<xacro:macro name="bumper_ctr_sensor">
+		<!-- I need this for contact sensor, "bumper sensor"  -->
+		<!-- I create this file in order to detect self-collisions and collisions with the ground  -->
+		<!-- This helps me to detect if the end effect touch the ground so I can reset the environment -->
 		<gazebo reference="shoulder_1_link">
-			<selfCollide>true</selfCollide>
+			<!-- contact sensor -->
 			<sensor name="shoulder_1_link_sensor" type="contact">
 				<selfCollide>true</selfCollide>
@@ -13,5 +14,6 @@
 					<collision>shoulder_1_collision</collision>
 				</contact>
-				<plugin name="bumper_shoulder_1" filename="libgazebo_ros_bumper.so">
+				<!-- gazebo plugin -->
+				<plugin name="gazebo_ros_bumper_sensor" filename="libgazebo_ros_bumper.so">
 					<ros>
 						<namespace>contact_sensor</namespace>
@@ -22,7 +24,6 @@
 			</sensor>
 		</gazebo>
-		<!-- Sensore su arm_1_link -->
 		<gazebo reference="arm_1_link">
-			<selfCollide>true</selfCollide>
+			<!-- contact sensor -->
 			<sensor name="arm_1_link_sensor" type="contact">
 				<selfCollide>true</selfCollide>
@@ -32,5 +33,6 @@
 					<collision>arm_1_link_collision</collision>
 				</contact>
-				<plugin name="bumper_arm_1" filename="libgazebo_ros_bumper.so">
+				<!-- gazebo plugin -->
+				<plugin name="gazebo_ros_bumper_sensor" filename="libgazebo_ros_bumper.so">
 					<ros>
 						<namespace>contact_sensor</namespace>
@@ -42,5 +44,5 @@
 		</gazebo>
 		<gazebo reference="arm_2_link">
-			<selfCollide>true</selfCollide>
+			<!-- contact sensor -->
 			<sensor name="arm_2_link_sensor" type="contact">
 				<selfCollide>true</selfCollide>
@@ -50,5 +52,6 @@
 					<collision>arm_2_link_collision</collision>
 				</contact>
-				<plugin name="bumper_arm_2" filename="libgazebo_ros_bumper.so">
+				<!-- gazebo plugin -->
+				<plugin name="gazebo_ros_bumper_sensor" filename="libgazebo_ros_bumper.so">
 					<ros>
 						<namespace>contact_sensor</namespace>
@@ -60,5 +63,5 @@
 		</gazebo>
 		<gazebo reference="wrist_1_link">
-			<selfCollide>true</selfCollide>
+			<!-- contact sensor -->
 			<sensor name="wrist_1_link_sensor" type="contact">
 				<selfCollide>true</selfCollide>
@@ -68,5 +71,6 @@
 					<collision>wrist_1_link_collision</collision>
 				</contact>
-				<plugin name="bumper_wrist_1" filename="libgazebo_ros_bumper.so">
+				<!-- gazebo plugin -->
+				<plugin name="gazebo_ros_bumper_sensor" filename="libgazebo_ros_bumper.so">
 					<ros>
 						<namespace>contact_sensor</namespace>
@@ -78,5 +82,5 @@
 		</gazebo>
 		<gazebo reference="wrist_2_link">
-			<selfCollide>true</selfCollide>
+			<!-- contact sensor -->
 			<sensor name="wrist_2_link_sensor" type="contact">
 				<selfCollide>true</selfCollide>
@@ -86,5 +90,6 @@
 					<collision>wrist_2_link_collision</collision>
 				</contact>
-				<plugin name="bumper_wrist_2" filename="libgazebo_ros_bumper.so">
+				<!-- gazebo plugin -->
+				<plugin name="gazebo_ros_bumper_sensor" filename="libgazebo_ros_bumper.so">
 					<ros>
 						<namespace>contact_sensor</namespace>
@@ -96,5 +101,5 @@
 		</gazebo>
 		<gazebo reference="wrist_3_link">
-			<selfCollide>true</selfCollide>
+			<!-- contact sensor -->
 			<sensor name="wrist_3_link_sensor" type="contact">
 				<selfCollide>true</selfCollide>
@@ -104,5 +109,6 @@
 					<collision>wrist_3_link_collision</collision>
 				</contact>
-				<plugin name="bumper_wrist_3" filename="libgazebo_ros_bumper.so">
+				<!-- gazebo plugin -->
+				<plugin name="gazebo_ros_bumper_sensor" filename="libgazebo_ros_bumper.so">
 					<ros>
 						<namespace>contact_sensor</namespace>

File: altri pacchetti/my_doosan_pkg/description/xacro/macro.internal_config_mod.xacro (robot description, xacro)
@@ -10,8 +10,4 @@
       <kp>1000000.0</kp>
       <kd>100.0</kd>
-      <mu1>30.0</mu1>
-      <mu2>30.0</mu2>
-      <maxVel>1.0</maxVel>
-      <minDepth>0.001</minDepth>
     </gazebo>
     <!-- Link1 -->
@@ -19,8 +15,4 @@
       <kp>1000000.0</kp>
       <kd>100.0</kd>
-      <mu1>30.0</mu1>
-      <mu2>30.0</mu2>
-      <maxVel>1.0</maxVel>
-      <minDepth>0.001</minDepth>
     </gazebo>
     <!-- Link2 -->

File: altri pacchetti/my_doosan_pkg/description/xacro/macro.tm5_900.xacro (robot description, xacro)
@@ -39,5 +39,5 @@
     wrist_3_lower_limit:=${-1.5*pi}    wrist_3_upper_limit:=${1.5*pi}
     transmission_hw_interface:=hardware_interface/PositionJointInterface
-    safety_limits:=true safety_pos_margin:=0.15
+    safety_limits:=false safety_pos_margin:=0.01
     safety_k_position:=20">
     <!-- Inertia parameters -->
